Commit message: rename vddben --> calvin inside files

File: vddben_description/bases/vddben_base.urdf.xacro (robot description, xacro)
@@ -3,5 +3,5 @@
   xmlns:interface="http://playerstage.sourceforge.net/gazebo/xmlschema/#interface"
   xmlns:xacro="http://ros.org/wiki/xacro"
-  name="vddben_base">
+  name="calvin_base">
   <xacro:property name="M_PI" value="3.1415926535897931" />
   <xacro:property name="wheel_width" value="0.06" />
@@ -56,5 +56,5 @@
   <!-- inertial measurement unit for gazebo -->
   <xacro:imu_gazebo link="base_link" imu_topic="imu" update_rate="100.0" stdev="${imu_stdev}" />
-  <xacro:macro name="vddben_wheel" params="name xyz rotate_visual">
+  <xacro:macro name="calvin_wheel" params="name xyz rotate_visual">
     <!-- rotate_visual: 0 for right side, 1 for left side -->
     <link name="${name}_wheel_link">
@@ -109,10 +109,10 @@
     </joint>
   </xacro:macro>
-  <xacro:vddben_wheel name="left_front" xyz="${wheel_x_offset} ${axis_length/2} ${wheel_z_offset}" rotate_visual="1" />
-  <xacro:vddben_wheel name="left_middle" xyz="0 ${axis_length/2} ${wheel_z_offset}" rotate_visual="1" />
-  <xacro:vddben_wheel name="left_rear" xyz="${-wheel_x_offset} ${axis_length/2} ${wheel_z_offset}" rotate_visual="1" />
-  <xacro:vddben_wheel name="right_front" xyz="${wheel_x_offset} ${-axis_length/2} ${wheel_z_offset}" rotate_visual="0" />
-  <xacro:vddben_wheel name="right_middle" xyz="0 ${-axis_length/2} ${wheel_z_offset}" rotate_visual="0" />
-  <xacro:vddben_wheel name="right_rear" xyz="${-wheel_x_offset} ${-axis_length/2} ${wheel_z_offset}" rotate_visual="0" />
+  <xacro:calvin_wheel name="left_front" xyz="${wheel_x_offset} ${axis_length/2} ${wheel_z_offset}" rotate_visual="1" />
+  <xacro:calvin_wheel name="left_middle" xyz="0 ${axis_length/2} ${wheel_z_offset}" rotate_visual="1" />
+  <xacro:calvin_wheel name="left_rear" xyz="${-wheel_x_offset} ${axis_length/2} ${wheel_z_offset}" rotate_visual="1" />
+  <xacro:calvin_wheel name="right_front" xyz="${wheel_x_offset} ${-axis_length/2} ${wheel_z_offset}" rotate_visual="0" />
+  <xacro:calvin_wheel name="right_middle" xyz="0 ${-axis_length/2} ${wheel_z_offset}" rotate_visual="0" />
+  <xacro:calvin_wheel name="right_rear" xyz="${-wheel_x_offset} ${-axis_length/2} ${wheel_z_offset}" rotate_visual="0" />
   <!-- base_footprint is a fictitious link(frame) that is on the ground right below base_link origin,
        navigation stack dedpends on this frame -->

File: vddben_description/robots/vddben.urdf.xacro (robot description, xacro)
@@ -2,6 +2,6 @@
 <robot
   xmlns:xacro="http://ros.org/wiki/xacro"
-  name="vddben">
-  <include filename="$(find vddben_description)/bases/vddben_base.urdf.xacro" />
-  <include filename="$(find vddben_description)/tops/muffin_top.urdf.xacro" />
+  name="calvin">
+  <include filename="$(find calvin_description)/bases/calvin_base.urdf.xacro" />
+  <include filename="$(find calvin_description)/tops/muffin_top.urdf.xacro" />
 </robot>
