Commit message: gazebo plugin controller added + collision box bug fixed

File: calvin_description/bases/calvin_base.urdf.xacro (robot description, xacro)
@@ -26,5 +26,5 @@
       <origin xyz="0 0 0" rpy="0 0 0" />
       <geometry>
-        <box size="1 1 1" />
+        <box size="0.55 0.32 0.155" />
       </geometry>
     </collision>
@@ -41,4 +41,24 @@
   <gazebo reference="base_link">
     <material value="Gazebo/Grey" />
+  </gazebo>
+  <gazebo>
+    <controller:gazebo_ros_kurt name="kurt_controller" plugin="libgazebo_ros_kurt.so">
+      <alwaysOn>true</alwaysOn>
+      <cmd_vel_topic_name>cmd_vel</cmd_vel_topic_name>
+      <odom_topic_name>odom</odom_topic_name>
+      <joint_states_topic_name>joint_states</joint_states_topic_name>
+      <left_front_wheel_joint>left_front_wheel_joint</left_front_wheel_joint>
+      <left_middle_wheel_joint>left_middle_wheel_joint</left_middle_wheel_joint>
+      <left_rear_wheel_joint>left_rear_wheel_joint</left_rear_wheel_joint>
+      <right_front_wheel_joint>right_front_wheel_joint</right_front_wheel_joint>
+      <right_middle_wheel_joint>right_middle_wheel_joint</right_middle_wheel_joint>
+      <right_rear_wheel_joint>right_rear_wheel_joint</right_rear_wheel_joint>
+      <wheel_separation>${axis_length}</wheel_separation>
+      <wheel_diameter>${2*wheel_radius}</wheel_diameter>
+      <turning_adaptation>${turning_adaptation}</turning_adaptation>
+      <torque>4.0</torque>
+      <max_velocity>0.9</max_velocity>
+      <updateRate>40.0</updateRate>
+    </controller:gazebo_ros_kurt>
   </gazebo>
   <!-- publish ground truth for pose of base_footprint -->

Commit message: added mesh for wheel type 1

File: calvin_description/bases/calvin_base.urdf.xacro (robot description, xacro)
@@ -81,7 +81,7 @@
       <visual>
         <origin xyz="0 0 0" rpy="${M_PI/2} 0 ${rotate_visual * M_PI}" />
-        <!--<origin xyz="0 0 0" rpy="0 0 ${rotate_visual * M_PI}" />-->
         <geometry>
-          <cylinder length="${wheel_width}" radius="${wheel_radius}"/>
+          <!--<cylinder length="${wheel_width}" radius="${wheel_radius}"/>-->
+          <mesh filename="package://calvin_description/meshes/wheel01.stl" />
         </geometry>
         <material name="blackish">
@@ -94,5 +94,6 @@
         <geometry>
           <!-- using STL for collision to fix http://answers.ros.org/question/2368/gazebo-model-wheels-slip-after-upgrade-to-electric -->
-          <cylinder length="${wheel_width}" radius="${wheel_radius}"/>
+          <!--<cylinder length="${wheel_width}" radius="${wheel_radius}"/>-->
+          <mesh filename="package://calvin_description/meshes/wheel01.stl" />
         </geometry>
       </collision>

Commit message: all geometry meshed

File: calvin_description/bases/calvin_base.urdf.xacro (robot description, xacro)
@@ -17,5 +17,6 @@
       <origin xyz="0 0 0" rpy="0 0 0" />
       <geometry>
-        <box size="0.55 0.32 0.155" />
+        <!--<box size="0.55 0.32 0.155" />-->
+        <mesh filename="package://calvin_description/meshes/item-base.stl"/>
       </geometry>
       <material name="grey" >
@@ -26,5 +27,6 @@
       <origin xyz="0 0 0" rpy="0 0 0" />
       <geometry>
-        <box size="0.55 0.32 0.155" />
+        <!--<box size="0.55 0.32 0.155" />-->
+        <mesh filename="package://calvin_description/meshes/item-base.stl"/>
       </geometry>
     </collision>
@@ -39,7 +41,7 @@
     </inertial>
   </link>
-  <gazebo reference="base_link">
-    <material value="Gazebo/Grey" />
-  </gazebo>
+  <!--<gazebo reference="base_link">-->
+    <!--<material value="Gazebo/Grey" />-->
+  <!--</gazebo>-->
   <gazebo>
     <controller:gazebo_ros_kurt name="kurt_controller" plugin="libgazebo_ros_kurt.so">
@@ -122,4 +124,5 @@
       <kd value="10000.0"/>
       <fdir1 value="1 0 0"/>  <!-- see http://answers.ros.org/question/607/rotation-error-in-gazebo-simulation -->
+      <material value="Gazebo/FlatBlack" />
     </gazebo>
     <joint name="${name}_wheel_joint" type="continuous">

File: calvin_description/tops/muffin_top.urdf.xacro (robot description, xacro)
@@ -4,5 +4,6 @@
     <visual>
       <geometry>
-        <box size="0.36 0.32 0.505" />
+        <!--<box size="0.36 0.32 0.505" />-->
+        <mesh filename="package://calvin_description/meshes/item-structure.stl"/>
       </geometry>
       <material name="grey" >
@@ -13,5 +14,6 @@
       <geometry>
         <!-- using STL for collision to fix http://answers.ros.org/question/2368/gazebo-model-wheels-slip-after-upgrade-to-electric -->
-        <box size="0.36 0.32 0.505" />
+        <!--<box size="0.36 0.32 0.505" />-->
+        <mesh filename="package://calvin_description/meshes/item-structure.stl"/>
       </geometry>
     </collision>
@@ -32,5 +34,6 @@
     <visual>
       <geometry>
-        <box size="0.02 0.02 1.4" />
+        <!--<box size="0.02 0.02 1.4" />-->
+        <mesh filename="package://calvin_description/meshes/item-pole.stl"/>
       </geometry>
       <material name="grey" >
@@ -41,5 +44,6 @@
       <geometry>
         <!-- using STL for collision to fix http://answers.ros.org/question/2368/gazebo-model-wheels-slip-after-upgrade-to-electric -->
-        <box size="0.02 0.02 1.4" />
+        <!--<box size="0.02 0.02 1.4" />-->
+        <mesh filename="package://calvin_description/meshes/item-pole.stl"/>
       </geometry>
     </collision>

Commit message: cleanup + sick tim + kinect + katana

File: calvin_description/bases/calvin_base.urdf.xacro (robot description, xacro)
@@ -41,7 +41,4 @@
     </inertial>
   </link>
-  <!--<gazebo reference="base_link">-->
-    <!--<material value="Gazebo/Grey" />-->
-  <!--</gazebo>-->
   <gazebo>
     <controller:gazebo_ros_kurt name="kurt_controller" plugin="libgazebo_ros_kurt.so">

File: calvin_description/robots/calvin.urdf.xacro (robot description, xacro)
@@ -5,4 +5,7 @@
   <include filename="$(find calvin_description)/bases/calvin_base.urdf.xacro" />
   <include filename="$(find calvin_description)/tops/muffin_top.urdf.xacro" />
+  <include filename="$(find calvin_description)/urdf/gazebo.urdf.xacro" />
+  <include filename="$(find sick_tim3xx)/urdf/sick_tim3xx.urdf.xacro" />
+  <xacro:sick_tim3xx laser_link="laser" />
   <joint name="laser_mount_joint" type="fixed">
     <origin xyz="0.25 0 0.08" rpy="0 0 0" />
@@ -10,5 +13,3 @@
     <child link="laser_mount_link" />
   </joint>
-  <include filename="$(find sick_tim3xx)/urdf/sick_tim3xx.urdf.xacro" />
-  <xacro:sick_tim3xx laser_link="laser" />
 </robot>

File: calvin_description/tops/muffin_top.urdf.xacro (robot description, xacro)
@@ -1,4 +1,22 @@
 <?xml version="1.0"?>
 <robot xmlns:xacro="http://ros.org/wiki/xacro">
+  <property name="sensor_mount_length" value="0.02" />
+  <property name="sensor_mount_width" value="0.139" />
+  <property name="sensor_mount_height" value="0.189" />
+  <property name="sensor_mount_mass" value="0.100" />
+  <property name="sensor_mount_x_offset" value="-0.16" />
+  <property name="kinect_fixture_length" value="0.02" />
+  <property name="kinect_fixture_width" value="0.02" />
+  <property name="kinect_fixture_height" value="0.265" />
+  <property name="kinect_fixture_mass" value="0.050" />
+  <property name="kinect_fixture_x_offset" value="0.00" />
+  <property name="kinect_fixture_joint_z_offset" value="-0.015" /> <!-- how much the joint center is displaced from the link center-->
+  <property name="laser_z_offset" value="-0.0407" />
+  <property name="kinect_x_offset" value="0.0" />
+  <property name="kinect_y_offset" value="0.05" />
+  <property name="kinect_z_offset" value="0.16" />
+  <property name="kinect_r" value="0.0" />
+  <property name="kinect_p" value="0.0" />
+  <property name="kinect_y" value="-0.07" />
   <link name="structure">
     <visual>
@@ -59,5 +77,79 @@
     <parent link="structure" />
     <child link="pole" />
-    <origin xyz="${-0.18 - 0.01} 0 ${0.4475 + 0.12}" rpy="0 0 0" />
+    <origin xyz="${-0.18 - 0.01} 0 0.2525" rpy="0 0 0" />
   </joint>
+  <!-- **************************** -->
+  <!-- *** Neuronics Katana Arm *** -->
+  <!-- **************************** -->
+  <include filename="$(find katana_description)/urdf/katana_450_6m90a_with_controlbox.urdf.xacro" />
+  <link name="katana_pattern"></link>
+  <joint name="katana_pattern_joint" type="fixed">
+    <parent link="katana_motor4_lift_link"/>
+    <child  link="katana_pattern" />
+    <origin xyz=".075 -.035 0.00" rpy="1.571 -1.571 0.151"/>
+  </joint>
+  <property name="baseplate_height" value="0.006" />
+  <joint name="kurtana_baseplate_controlbox_joint" type="fixed">
+    <parent link="structure" />
+    <child link="katana_internal_controlbox_link" />
+    <origin xyz="0 0 ${baseplate_height*1.5 + 0.2525}" rpy="0 0 0" />
+  </joint>
+  <!-- ********************************** -->
+  <!-- *** Kinect / Xtion RGBD Camera *** -->
+  <!-- ********************************** -->
+  <joint name="kinect_stretch_joint" type="prismatic">
+    <parent link="pole" />
+    <child link="kurtana_stretch_link" />
+    <origin xyz="0 0 0.5" rpy="0 0 0"/>
+    <axis xyz="0 0 1"/>
+    <limit effort="1000.0" lower="${-M_PI/2}" upper="${M_PI/2}" velocity="2.0"/>
+  </joint>
+  <joint name="kinect_pitch_joint" type="revolute">
+    <parent link="kurtana_stretch_link" />
+    <child link="kurtana_pitch_link" />
+    <origin xyz="0 0 0" rpy="0 0 0"/>
+    <axis xyz="0 1 0"/>
+    <limit effort="1000.0" lower="${-M_PI/2}" upper="${M_PI/2}" velocity="2.0"/>
+  </joint>
+  <joint name="kinect_yaw_joint" type="revolute">
+    <parent link="kurtana_pitch_link" />
+    <child link="kurtana_yaw_link" />
+    <origin xyz="0 0 0" rpy="0 0 0"/>
+    <axis xyz="0 1 0"/>
+    <limit effort="1000.0" lower="${-M_PI/2}" upper="${M_PI/2}" velocity="2.0"/>
+  </joint>
+  <include filename="$(find kurt_description)/parts/kinect.urdf.xacro" />
+  <xacro:kinect camera="kinect" />
+  <joint name="calvin_kinect_joint" type="fixed">
+    <parent link="kurtana_pitchpole_link" />
+    <child  link="kinect_link" />
+    <origin xyz="0.1 0 0.5" rpy="0 0.5 0"/>
+  </joint>
+  <link name="kurtana_pitchpole_link">
+    <visual>
+      <origin rpy="${-M_PI/2} 0 0" xyz="0 0 0"/>
+      <geometry>
+        <cylinder radius="${pitchpole_radius}" length="${pitchpole_length}"/>
+      </geometry>
+      <material name="grey" />
+    </visual>
+    <collision>
+      <origin rpy="${-M_PI/2} 0 0" xyz="0 0 0"/>
+      <geometry>
+        <cylinder radius="${pitchpole_radius}" length="${pitchpole_length}"/>
+      </geometry>
+    </collision>
+    <xacro:cylinder_inertial radius="${pitchpole_radius}" length="${pitchpole_length}" mass="${pitchpole_mass}" />
+  </link>
+  <xacro:macro name="kinect_pole_transmission" params="name">
+    <transmission name="${name}_trans" type="pr2_mechanism_model/SimpleTransmission">
+      <actuator name="${name}_motor" />
+      <joint name="${name}_joint" />
+      <mechanicalReduction>1</mechanicalReduction>
+      <motorTorqueConstant>1</motorTorqueConstant>
+    </transmission>
+  </xacro:macro>
+  <xacro:kinect_pole_transmission name="kinect_stretch" />
+  <xacro:kinect_pole_transmission name="kinect_roll" />
+  <xacro:kinect_pole_transmission name="kinect_pitch" />
 </robot>
