Commit message: added but did not completely made working the following: robot_state_publisher calvin_joint_commander imu to real calvin usb_cam for logitech vga webcam openni for xtion

File: calvin_description/urdf/calvin.urdf.xacro (robot description, xacro)
@@ -1,4 +1,6 @@
 <?xml version="1.0"?>
-<robot xmlns:xacro="http://ros.org/wiki/xacro">
+<robot xmlns:xacro="http://ros.org/wiki/xacro"
+  xmlns:sensor="http://playerstage.sourceforge.net/gazebo/xmlschema/#sensor"
+  xmlns:controller="http://playerstage.sourceforge.net/gazebo/xmlschema/#controller">
   <property name="sensor_mount_length" value="0.02" />
   <property name="sensor_mount_width" value="0.139" />
@@ -70,4 +72,63 @@
     <origin xyz="${-0.18 - 0.01} 0 0.2525" rpy="0 0 0" />
   </joint>
+  <!-- ******************************** -->
+  <!-- *** gazebo ros camera plugin *** -->
+  <!-- ******************************** -->
+  <xacro:macro name="webcam" params="">
+    <gazebo reference="webcam">
+      <sensor:camera name="webcam">
+        <imageFormat>L8</imageFormat>
+        <imageSize>640 480</imageSize>
+        <hfov>57</hfov>
+        <nearClip>0.01</nearClip>
+        <farClip>5</farClip>
+        <updateRate>1.0</updateRate>
+        <baseline>0.2</baseline>
+        <controller:gazebo_ros_camera name="webcam_controller" plugin="libgazebo_ros_camera.so">
+          <robotNamespace>webcam</robotNamespace>
+          <imageTopicName>image_raw</imageTopicName>
+          <cameraInfoTopicName>camera_info</cameraInfoTopicName>
+          <cameraName>webcam</cameraName>
+          <frameName>/world</frameName>
+          <updateRate>1</updateRate>
+          <CxPrime>10</CxPrime>
+          <Cx>10</Cx>
+          <Cy>10</Cy>
+          <focalLength>10</focalLength>
+          <hackBaseline>10</hackBaseline>
+          <distortionK1>0</distortionK1>
+          <distortionK2>0</distortionK2>
+          <distortionK3>0</distortionK3>
+          <distortionT1>0</distortionT1>
+          <distortionT2>0</distortionT2>
+        </controller:gazebo_ros_camera>
+      </sensor:camera>
+      <material value="Gazebo/Red" />
+    </gazebo>
+    <link name="webcam_link">
+      <visual>
+        <origin rpy="0 0 0" xyz="0 0 0"/>
+        <geometry>
+          <box size="0.1 0.1 0.1" />
+        </geometry>
+        <material name="red">
+          <color rgba="1 0 0 1" />
+        </material>
+      </visual>
+      <collision>
+        <origin rpy="0 0 0" xyz="0 0 0"/>
+        <geometry>
+          <box size="0.1 0.1 0.1" />
+        </geometry>
+      </collision>
+      <xacro:box_inertial x="0.1" y="0.1" z="0.1" mass="0.01"/>
+    </link>
+    <joint name="webcam_joint" type="fixed">
+      <origin xyz="0 0 0" rpy="0 0 0" />
+      <parent link="pole" />
+      <child link="webcam_link" />
+    </joint>
+  </xacro:macro>
+  <xacro:webcam/>
   <!-- **************************** -->
   <!-- *** Neuronics Katana Arm *** -->

Commit message: launch file and urdf update + joint commander. first rosbag.

File: calvin_description/urdf/calvin.urdf.xacro (robot description, xacro)
@@ -51,5 +51,5 @@
     <visual>
       <geometry>
-        <!--<box size="0.02 0.02 1.4" />-->
+        <!--<box size="0.02 0.02 1.0" />-->
         <mesh filename="package://calvin_description/meshes/item-pole.stl"/>
       </geometry>
@@ -61,14 +61,14 @@
       <geometry>
         <!-- using STL for collision to fix http://answers.ros.org/question/2368/gazebo-model-wheels-slip-after-upgrade-to-electric -->
-        <!--<box size="0.02 0.02 1.4" />-->
+        <!--<box size="0.02 0.02 1.0" />-->
         <mesh filename="package://calvin_description/meshes/item-pole.stl"/>
       </geometry>
     </collision>
-    <xacro:box_inertial x="0.02" y="0.02" z="1.4" mass="0.25"/>
+    <xacro:box_inertial x="0.02" y="0.02" z="1.0" mass="0.25"/>
   </link>
   <joint name="structure_to_pole_joint" type="fixed">
     <parent link="structure" />
     <child link="pole" />
-    <origin xyz="${-0.18 - 0.01} 0 0.2525" rpy="0 0 0" />
+    <origin xyz="${-0.18 - 0.01} 0 ${0.5 + 0.2525 + 0.005}" rpy="0 0 0" />
   </joint>
   <!-- ******************************** -->
@@ -154,8 +154,8 @@
       <origin rpy="0 0 0" xyz="0 0 0"/>
       <geometry>
-        <box size="0.046 0.06 0.02" />
+        <box size="0.08 0.06 0.02" />
       </geometry>
-      <material name="red">
-        <color rgba="1 0 0 1" />
+      <material name="grey">
+        <color rgba="0.5 0.5 0.5 1" />
       </material>
     </visual>
@@ -163,39 +163,14 @@
       <origin rpy="0 0 0" xyz="0 0 0"/>
       <geometry>
-        <box size="0.046 0.06 0.02" />
+        <box size="0.08 0.06 0.02" />
       </geometry>
     </collision>
-    <xacro:box_inertial x="0.1" y="0.1" z="0.1" mass="0.01"/>
+    <xacro:box_inertial x="0.08" y="0.06" z="0.02" mass="0.01"/>
   </link>
   <joint name="kinect_pitch_joint" type="revolute">
     <parent link="pole" />
     <child link="kinect_pitch_link" />
-    <origin xyz="0.05 0 0.5" rpy="0 0 0"/>
+    <origin xyz="0.025 0 0.46" rpy="0 0 0"/>
     <axis xyz="0 1 0"/>
-    <limit effort="1000.0" lower="${-M_PI/2}" upper="${M_PI/2}" velocity="2.0"/>
-  </joint>
-  <link name="kinect_yaw_link">
-    <visual>
-      <origin rpy="0 0 0" xyz="0 0 0"/>
-      <geometry>
-        <box size="0.01 0.1 0.01" />
-      </geometry>
-      <material name="green" >
-        <color rgba="0 1 0 1" />
-      </material>
-    </visual>
-    <collision>
-      <origin rpy="0 0 0" xyz="0 0 0"/>
-      <geometry>
-        <box size="0.1 0.1 0.1" />
-      </geometry>
-    </collision>
-    <xacro:box_inertial x="0.1" y="0.1" z="0.1" mass="0.1"/>
-  </link>
-  <joint name="kinect_yaw_joint" type="revolute">
-    <parent link="kinect_pitch_link" />
-    <child link="kinect_yaw_link" />
-    <origin xyz="0.05 0 0" rpy="0 0 0"/>
-    <axis xyz="0 0 1"/>
     <limit effort="1000.0" lower="${-M_PI/2}" upper="${M_PI/2}" velocity="2.0"/>
   </joint>
@@ -203,7 +178,7 @@
   <xacro:kinect camera="kinect" />
   <joint name="calvin_kinect_joint" type="fixed">
-    <parent link="kinect_yaw_link" />
+    <parent link="kinect_pitch_link" />
     <child  link="kinect_link" />
-    <origin xyz="0.05 0 0" rpy="0 0.5 0"/>
+    <origin xyz="0.03 0.03 0.02" rpy="0 0 0"/>
   </joint>
   <xacro:macro name="kinect_pole_transmission" params="name">
@@ -216,4 +191,3 @@
   </xacro:macro>
   <xacro:kinect_pole_transmission name="kinect_pitch" />
-  <xacro:kinect_pole_transmission name="kinect_yaw" />
 </robot>

Commit message: adjusted camera position in urdf

File: calvin_description/urdf/calvin.urdf.xacro (robot description, xacro)
@@ -104,14 +104,14 @@
         </controller:gazebo_ros_camera>
       </sensor:camera>
-      <material value="Gazebo/Red" />
+      <material value="Gazebo/Gray" />
     </gazebo>
     <link name="webcam_link">
       <visual>
-        <origin rpy="0 0 0" xyz="0 0 0"/>
+        <origin rpy="0 0 0" xyz="-0.015 0 0"/>
         <geometry>
-          <box size="0.1 0.1 0.1" />
+          <box size="0.025 0.038 0.038" />
         </geometry>
-        <material name="red">
-          <color rgba="1 0 0 1" />
+        <material name="gray">
+          <color rgba="0.4 0.4 0.4 1" />
         </material>
       </visual>
@@ -119,5 +119,5 @@
         <origin rpy="0 0 0" xyz="0 0 0"/>
         <geometry>
-          <box size="0.1 0.1 0.1" />
+          <box size="0.03 0.04 0.04" />
         </geometry>
       </collision>
@@ -125,5 +125,5 @@
     </link>
     <joint name="webcam_joint" type="fixed">
-      <origin xyz="0 0 0" rpy="0 0 0" />
+      <origin xyz="0.07 0 0.35" rpy="0 0.1 0" />
       <parent link="pole" />
       <child link="webcam_link" />

Commit message: optical frame for webcam

File: calvin_description/urdf/calvin.urdf.xacro (robot description, xacro)
@@ -107,19 +107,4 @@
     </gazebo>
     <link name="webcam_link">
-      <visual>
-        <origin rpy="0 0 0" xyz="-0.015 0 0"/>
-        <geometry>
-          <box size="0.025 0.038 0.038" />
-        </geometry>
-        <material name="gray">
-          <color rgba="0.4 0.4 0.4 1" />
-        </material>
-      </visual>
-      <collision>
-        <origin rpy="0 0 0" xyz="0 0 0"/>
-        <geometry>
-          <box size="0.03 0.04 0.04" />
-        </geometry>
-      </collision>
       <xacro:box_inertial x="0.1" y="0.1" z="0.1" mass="0.01"/>
     </link>
@@ -128,4 +113,12 @@
       <parent link="pole" />
       <child link="webcam_link" />
+    </joint>
+    <link name="webcam_optical_link">
+      <xacro:box_inertial x="0.1" y="0.1" z="0.1" mass="0.01"/>
+    </link>
+    <joint name="webcam_optical_joint" type="fixed">
+      <origin xyz="0 0 0" rpy="${-M_PI/2} 0 ${-M_PI/2}" />
+      <parent link="webcam_link" />
+      <child link="webcam_optical_link" />
     </joint>
   </xacro:macro>

Commit message: fine tuning of calvin urdf. added some parameters.

File: calvin_description/urdf/calvin.urdf.xacro (robot description, xacro)
@@ -21,11 +21,15 @@
   <property name="kinect_p" value="0.0" />
   <property name="kinect_y" value="-0.07" />
-  <property name="pitchpole_radius" value="0.012"/>
-  <property name="pitchpole_length" value="0.23"/>
-  <property name="pitchpole_mass" value="0.050"/>
+  <xacro:property name="pole_length" value="0.02"/>
+  <xacro:property name="pole_width" value="0.02"/>
+  <xacro:property name="pole_height" value="1"/>
+  <xacro:property name="structure_length" value="0.36"/>
+  <xacro:property name="structure_width" value="0.32"/>
+  <xacro:property name="structure_height" value="0.51"/>
+  <xacro:property name="item_width" value="0.02"/>
   <link name="structure">
     <visual>
       <geometry>
-        <!--<box size="0.36 0.32 0.505" />-->
+        <!--<box size="${structure_length} ${structure_width} ${structure_height}" />-->
         <mesh filename="package://calvin_description/meshes/item-structure.stl"/>
       </geometry>
@@ -37,19 +41,19 @@
       <geometry>
         <!-- using STL for collision to fix http://answers.ros.org/question/2368/gazebo-model-wheels-slip-after-upgrade-to-electric -->
-        <!--<box size="0.36 0.32 0.505" />-->
+        <!--<box size="${structure_length} ${structure_width} ${structure_height}" />-->
         <mesh filename="package://calvin_description/meshes/item-structure.stl"/>
       </geometry>
     </collision>
-    <xacro:box_inertial x="0.36" y="0.32" z="0.505" mass="2"/>
+    <xacro:box_inertial x="${structure_length}" y="${structure_width}" z="${structure_height}" mass="2"/>
   </link>
   <joint name="top_to_structure" type="fixed">
     <parent link="base_link" />
     <child link="structure" />
-    <origin xyz="${0.095 - 0.02} 0 ${0.2525 + 0.0775}" rpy="0 0 0" />
+    <origin xyz="${base_link_length/2 - structure_length/2 - item_width} 0 ${structure_height/2 + base_link_height/2}" rpy="0 0 0" />
   </joint>
   <link name="pole">
     <visual>
       <geometry>
-        <!--<box size="0.02 0.02 1.0" />-->
+        <!--<box size="${pole_length} ${pole_width} ${pole_height}" />-->
         <mesh filename="package://calvin_description/meshes/item-pole.stl"/>
       </geometry>
@@ -61,14 +65,14 @@
       <geometry>
         <!-- using STL for collision to fix http://answers.ros.org/question/2368/gazebo-model-wheels-slip-after-upgrade-to-electric -->
-        <!--<box size="0.02 0.02 1.0" />-->
+        <!--<box size="${pole_length} ${pole_width} ${pole_height}" />-->
         <mesh filename="package://calvin_description/meshes/item-pole.stl"/>
       </geometry>
     </collision>
-    <xacro:box_inertial x="0.02" y="0.02" z="1.0" mass="0.25"/>
+    <xacro:box_inertial x="${pole_length}" y="${pole_width}" z="${pole_height}" mass="0.25"/>
   </link>
   <joint name="structure_to_pole_joint" type="fixed">
     <parent link="structure" />
     <child link="pole" />
-    <origin xyz="${-0.18 - 0.01} 0 ${0.5 + 0.2525 + 0.005}" rpy="0 0 0" />
+    <origin xyz="${-structure_length/2 - pole_length/2} 0 ${pole_height/2 + structure_height/2}" rpy="0 0 0" />
   </joint>
   <!-- ******************************** -->
@@ -110,5 +114,5 @@
     </link>
     <joint name="webcam_joint" type="fixed">
-      <origin xyz="0.07 0 0.35" rpy="0 0.1 0" />
+      <origin xyz="0.07 0 0.315" rpy="0 0.1 0" />
       <parent link="pole" />
       <child link="webcam_link" />
@@ -184,3 +188,20 @@
   </xacro:macro>
   <xacro:kinect_pole_transmission name="kinect_pitch" />
+  <link name="test">
+    <visual>
+      <origin xyz="0 0 0" rpy="0 0 0" />
+      <geometry>
+        <box size="0.55 0.32 ${1.72 * 2}" />
+      </geometry>
+      <material name="red" >
+        <color rgba="1 0 0 1" />
+      </material>
+    </visual>
+  </link>
+  <joint name="test_joint" type="fixed">
+    <origin xyz="0 0 0" rpy="0 0 0" />
+    <parent link="base_footprint"/>
+    <child link="test"/>
+    <axis xyz="0 0 0"/>
+  </joint>
 </robot>

Commit message: fine tuning for kinect and webcam

File: calvin_description/urdf/calvin.urdf.xacro (robot description, xacro)
@@ -28,4 +28,12 @@
   <xacro:property name="structure_height" value="0.51"/>
   <xacro:property name="item_width" value="0.02"/>
+  <xacro:property name="webcam_pitch_link_length" value="0.082"/>
+  <xacro:property name="webcam_pitch_link_width" value="0.095"/>
+  <xacro:property name="webcam_pitch_link_height" value="0.02"/>
+  <xacro:property name="webcam_z_offset" value="0.315"/>
+  <xacro:property name="kinect_pitch_link_length" value="0.08"/>
+  <xacro:property name="kinect_pitch_link_width" value="0.17"/>
+  <xacro:property name="kinect_pitch_link_height" value="0.02"/>
+  <xacro:property name="kinect_pitch_link_z_offset" value="0.46"/>
   <link name="structure">
     <visual>
@@ -110,10 +118,47 @@
       <material value="Gazebo/Gray" />
     </gazebo>
+    <link name="webcam_pitch_link">
+      <visual>
+        <origin rpy="0 0 0" xyz="${webcam_pitch_link_length/2 - item_width/2} 0 -${webcam_pitch_link_height}"/>
+        <geometry>
+          <box size="${webcam_pitch_link_length} ${webcam_pitch_link_width} ${webcam_pitch_link_height}" />
+        </geometry>
+        <material name="grey" >
+          <color rgba="0.5 0.5 0.5 1" />
+        </material>
+      </visual>
+      <collision>
+        <geometry>
+          <box size="${webcam_pitch_link_length} ${webcam_pitch_link_width} ${webcam_pitch_link_height}" />
+        </geometry>
+      </collision>
+      <xacro:box_inertial x="${webcam_pitch_link_length}" y="${webcam_pitch_link_width}" z="${webcam_pitch_link_height}" mass="0.01"/>
+    </link>
+    <joint name="webcam_pitch_joint" type="revolute">
+      <origin xyz="0 0 ${webcam_z_offset}" rpy="0 0 0" />
+      <parent link="pole" />
+      <child link="webcam_pitch_link" />
+      <axis xyz="0 1 0"/>
+      <limit effort="1000.0" lower="${-M_PI/2}" upper="${M_PI/2}" velocity="2.0"/>
+    </joint>
     <link name="webcam_link">
+      <visual>
+        <geometry>
+          <box size="0.02 0.085 0.02" />
+        </geometry>
+        <material name="black" >
+          <color rgba="0 0 0 1" />
+        </material>
+      </visual>
+      <collision>
+        <geometry>
+          <box size="0.02 0.085 0.02" />
+        </geometry>
+      </collision>
       <xacro:box_inertial x="0.1" y="0.1" z="0.1" mass="0.01"/>
     </link>
     <joint name="webcam_joint" type="fixed">
-      <origin xyz="0.07 0 0.315" rpy="0 0.1 0" />
-      <parent link="pole" />
+      <origin xyz="0.06 0 -0.04" rpy="0 0 0" />
+      <parent link="webcam_pitch_link" />
       <child link="webcam_link" />
     </joint>
@@ -149,7 +194,7 @@
   <link name="kinect_pitch_link">
     <visual>
-      <origin rpy="0 0 0" xyz="0 0 0"/>
-      <geometry>
-        <box size="0.08 0.06 0.02" />
+      <origin rpy="${kinect_pitch_link_length/2 - item_width/2} 0 0" xyz="0 0 0"/>
+      <geometry>
+        <box size="${kinect_pitch_link_length} ${kinect_pitch_link_width} ${kinect_pitch_link_height}" />
       </geometry>
       <material name="grey">
@@ -158,15 +203,15 @@
     </visual>
     <collision>
-      <origin rpy="0 0 0" xyz="0 0 0"/>
-      <geometry>
-        <box size="0.08 0.06 0.02" />
+      <origin rpy="${kinect_pitch_link_length/2 - item_width/2} 0 0" xyz="0 0 0"/>
+      <geometry>
+        <box size="${kinect_pitch_link_length} ${kinect_pitch_link_width} ${kinect_pitch_link_height}" />
       </geometry>
     </collision>
-    <xacro:box_inertial x="0.08" y="0.06" z="0.02" mass="0.01"/>
+    <xacro:box_inertial x="${kinect_pitch_link_length}" y="${kinect_pitch_link_width}" z="${kinect_pitch_link_height}" mass="0.01"/>
   </link>
   <joint name="kinect_pitch_joint" type="revolute">
     <parent link="pole" />
     <child link="kinect_pitch_link" />
-    <origin xyz="0.025 0 0.46" rpy="0 0 0"/>
+    <origin xyz="0 0 ${kinect_pitch_link_z_offset}" rpy="0 0 0"/>
     <axis xyz="0 1 0"/>
     <limit effort="1000.0" lower="${-M_PI/2}" upper="${M_PI/2}" velocity="2.0"/>
@@ -188,20 +233,3 @@
   </xacro:macro>
   <xacro:kinect_pole_transmission name="kinect_pitch" />
-  <link name="test">
-    <visual>
-      <origin xyz="0 0 0" rpy="0 0 0" />
-      <geometry>
-        <box size="0.55 0.32 ${1.72 * 2}" />
-      </geometry>
-      <material name="red" >
-        <color rgba="1 0 0 1" />
-      </material>
-    </visual>
-  </link>
-  <joint name="test_joint" type="fixed">
-    <origin xyz="0 0 0" rpy="0 0 0" />
-    <parent link="base_footprint"/>
-    <child link="test"/>
-    <axis xyz="0 0 0"/>
-  </joint>
 </robot>

Commit message: calvin urdf: Added imu link and joint.
calvin_description: added imu link and joint to calvin.urdf.xacro
calvin_bringup: removed static transform publisher entry of imu in ekf.launch

File: calvin_description/urdf/calvin.urdf.xacro (robot description, xacro)
@@ -60,4 +60,10 @@
     <origin xyz="${base_link_length/2 - structure_length/2 - item_width} 0 ${structure_height/2 + base_link_height/2}" rpy="0 0 0" />
   </joint>
+  <link name="imu" />
+  <joint name="structure_to_imu_joint" type="fixed">
+    <parent link="base_link" />
+    <child link="imu" />
+    <origin xyz="0 0 0" rpy="0 0 0" />
+  </joint>
   <link name="pole">
     <visual>

Commit message: Fix tf frame of imu

File: calvin_description/urdf/calvin.urdf.xacro (robot description, xacro)
@@ -64,5 +64,5 @@
     <parent link="base_link" />
     <child link="imu" />
-    <origin xyz="0 0 0" rpy="0 0 0" />
+    <origin xyz="0 0 0" rpy="${M_PI} 0 ${M_PI}" />
   </joint>
   <link name="pole">

Commit message: finetuning of kinect fixture

File: calvin_description/urdf/calvin.urdf.xacro (robot description, xacro)
@@ -3,22 +3,7 @@
   xmlns:sensor="http://playerstage.sourceforge.net/gazebo/xmlschema/#sensor"
   xmlns:controller="http://playerstage.sourceforge.net/gazebo/xmlschema/#controller">
-  <property name="sensor_mount_length" value="0.02" />
-  <property name="sensor_mount_width" value="0.139" />
-  <property name="sensor_mount_height" value="0.189" />
-  <property name="sensor_mount_mass" value="0.100" />
-  <property name="sensor_mount_x_offset" value="-0.16" />
-  <property name="kinect_fixture_length" value="0.02" />
-  <property name="kinect_fixture_width" value="0.02" />
-  <property name="kinect_fixture_height" value="0.265" />
-  <property name="kinect_fixture_mass" value="0.050" />
-  <property name="kinect_fixture_x_offset" value="0.00" />
-  <property name="kinect_fixture_joint_z_offset" value="-0.015" /> <!-- how much the joint center is displaced from the link center-->
-  <property name="laser_z_offset" value="-0.0407" />
-  <property name="kinect_x_offset" value="0.0" />
-  <property name="kinect_y_offset" value="0.05" />
-  <property name="kinect_z_offset" value="0.16" />
-  <property name="kinect_r" value="0.0" />
-  <property name="kinect_p" value="0.0" />
-  <property name="kinect_y" value="-0.07" />
+  <property name="kinect_x_offset" value="0.06" />
+  <property name="kinect_y_offset" value="0.03" />
+  <property name="kinect_z_offset" value="0.05" />
   <xacro:property name="pole_length" value="0.02"/>
   <xacro:property name="pole_width" value="0.02"/>
@@ -200,5 +185,5 @@
   <link name="kinect_pitch_link">
     <visual>
-      <origin rpy="${kinect_pitch_link_length/2 - item_width/2} 0 0" xyz="0 0 0"/>
+      <origin xyz="${kinect_pitch_link_length/2 - item_width/2} 0 0" rpy="0 0 0"/>
       <geometry>
         <box size="${kinect_pitch_link_length} ${kinect_pitch_link_width} ${kinect_pitch_link_height}" />
@@ -209,5 +194,5 @@
     </visual>
     <collision>
-      <origin rpy="${kinect_pitch_link_length/2 - item_width/2} 0 0" xyz="0 0 0"/>
+      <origin xyz="${kinect_pitch_link_length/2 - item_width/2} 0 0" rpy="0 0 0"/>
       <geometry>
         <box size="${kinect_pitch_link_length} ${kinect_pitch_link_width} ${kinect_pitch_link_height}" />
@@ -228,5 +213,5 @@
     <parent link="kinect_pitch_link" />
     <child  link="kinect_link" />
-    <origin xyz="0.03 0.03 0.02" rpy="0 0 0"/>
+    <origin xyz="${kinect_x_offset} ${kinect_y_offset} ${kinect_z_offset}" rpy="0 0 0"/>
   </joint>
   <xacro:macro name="kinect_pole_transmission" params="name">

Commit message: vgacamera calibration done

File: calvin_description/urdf/calvin.urdf.xacro (robot description, xacro)
@@ -150,5 +150,5 @@
     </link>
     <joint name="webcam_joint" type="fixed">
-      <origin xyz="0.06 0 -0.04" rpy="0 0 0" />
+      <origin xyz="0.06 0.01 -0.04" rpy="0 0 0" />
       <parent link="webcam_pitch_link" />
       <child link="webcam_link" />
