Commit message: sick laserscanner added

File: calvin_description/robots/calvin.urdf.xacro (robot description, xacro)
@@ -5,3 +5,10 @@
   <include filename="$(find calvin_description)/bases/calvin_base.urdf.xacro" />
   <include filename="$(find calvin_description)/tops/muffin_top.urdf.xacro" />
+  <joint name="laser_mount_joint" type="fixed">
+    <origin xyz="0.25 0 0.08" rpy="0 0 0" />
+    <parent link="base_link"/>
+    <child link="laser_mount_link" />
+  </joint>
+  <include filename="$(find sick_tim3xx)/urdf/sick_tim3xx.urdf.xacro" />
+  <xacro:sick_tim3xx laser_link="laser" />
 </robot>

Commit message: intertials renaming fixing

File: calvin_description/robots/calvin.urdf.xacro (robot description, xacro)
@@ -3,7 +3,11 @@
   xmlns:xacro="http://ros.org/wiki/xacro"
   name="calvin">
-  <include filename="$(find calvin_description)/bases/calvin_base.urdf.xacro" />
-  <include filename="$(find calvin_description)/tops/muffin_top.urdf.xacro" />
-  <include filename="$(find calvin_description)/urdf/gazebo.urdf.xacro" />
+  I
+  <xacro:property name="imu_stdev" value="0.00017" />
+  <include filename="$(find volksbot_driver)/urdf/volksbot.urdf.xacro" />
+  <include filename="$(find calvin_description)/urdf/muffinsetup.urdf.xacro" />
+  <!--<include filename="$(find calvin_description)/urdf/gazebo.urdf.xacro" />-->
+  <!-- inertial measurement unit for gazebo -->
+  <xacro:imu_gazebo link="base_link" imu_topic="imu" update_rate="100.0" stdev="${imu_stdev}" />
   <include filename="$(find sick_tim3xx)/urdf/sick_tim3xx.urdf.xacro" />
   <xacro:sick_tim3xx laser_link="laser" />

File: calvin_description/urdf/muffinsetup.urdf.xacro (robot description, xacro)
@@ -19,4 +19,7 @@
   <property name="kinect_p" value="0.0" />
   <property name="kinect_y" value="-0.07" />
+  <property name="pitchpole_radius" value="0.012"/>
+  <property name="pitchpole_length" value="0.23"/>
+  <property name="pitchpole_mass" value="0.050"/>
   <link name="structure">
     <visual>
@@ -36,11 +39,5 @@
       </geometry>
     </collision>
-    <inertial>
-      <mass value="1.0" />
-      <origin xyz="-0.005401183 0.0 0.141356018" />
-      <inertia ixx="0.022277280" ixy="-0.000000004" ixz="-0.001009999"
-        iyy="0.017783837" iyz="0.0"
-        izz="0.025523417" />
-    </inertial>
+    <xacro:box_inertial x="0.36" y="0.32" z="0.505" mass="2"/>
   </link>
   <joint name="top_to_structure" type="fixed">
@@ -66,13 +63,7 @@
       </geometry>
     </collision>
-    <inertial>
-      <mass value="0.5" />
-      <origin xyz="-0.005401183 0.0 0.141356018" />
-      <inertia ixx="0.022277280" ixy="-0.000000004" ixz="-0.001009999"
-        iyy="0.017783837" iyz="0.0"
-        izz="0.025523417" />
-    </inertial>
+    <xacro:box_inertial x="0.02" y="0.02" z="1.4" mass="0.25"/>
   </link>
-  <joint name="structure_to_pole" type="fixed">
+  <joint name="structure_to_pole_joint" type="fixed">
     <parent link="structure" />
     <child link="pole" />
@@ -98,48 +89,61 @@
   <!-- *** Kinect / Xtion RGBD Camera *** -->
   <!-- ********************************** -->
-  <joint name="kinect_stretch_joint" type="prismatic">
+  <link name="kinect_pitch_link">
+    <visual>
+      <origin rpy="0 0 0" xyz="0 0 0"/>
+      <geometry>
+        <box size="0.046 0.06 0.02" />
+      </geometry>
+      <material name="red">
+        <color rgba="1 0 0 1" />
+      </material>
+    </visual>
+    <collision>
+      <origin rpy="0 0 0" xyz="0 0 0"/>
+      <geometry>
+        <box size="0.046 0.06 0.02" />
+      </geometry>
+    </collision>
+    <xacro:box_inertial x="0.1" y="0.1" z="0.1" mass="0.01"/>
+  </link>
+  <joint name="kinect_pitch_joint" type="revolute">
     <parent link="pole" />
-    <child link="kurtana_stretch_link" />
-    <origin xyz="0 0 0.5" rpy="0 0 0"/>
+    <child link="kinect_pitch_link" />
+    <origin xyz="0.05 0 0.5" rpy="0 0 0"/>
+    <axis xyz="0 1 0"/>
+    <limit effort="1000.0" lower="${-M_PI/2}" upper="${M_PI/2}" velocity="2.0"/>
+  </joint>
+  <link name="kinect_yaw_link">
+    <visual>
+      <origin rpy="0 0 0" xyz="0 0 0"/>
+      <geometry>
+        <box size="0.01 0.1 0.01" />
+      </geometry>
+      <material name="green" >
+        <color rgba="0 1 0 1" />
+      </material>
+    </visual>
+    <collision>
+      <origin rpy="0 0 0" xyz="0 0 0"/>
+      <geometry>
+        <box size="0.1 0.1 0.1" />
+      </geometry>
+    </collision>
+    <xacro:box_inertial x="0.1" y="0.1" z="0.1" mass="0.1"/>
+  </link>
+  <joint name="kinect_yaw_joint" type="revolute">
+    <parent link="kinect_pitch_link" />
+    <child link="kinect_yaw_link" />
+    <origin xyz="0.05 0 0" rpy="0 0 0"/>
     <axis xyz="0 0 1"/>
     <limit effort="1000.0" lower="${-M_PI/2}" upper="${M_PI/2}" velocity="2.0"/>
   </joint>
-  <joint name="kinect_pitch_joint" type="revolute">
-    <parent link="kurtana_stretch_link" />
-    <child link="kurtana_pitch_link" />
-    <origin xyz="0 0 0" rpy="0 0 0"/>
-    <axis xyz="0 1 0"/>
-    <limit effort="1000.0" lower="${-M_PI/2}" upper="${M_PI/2}" velocity="2.0"/>
-  </joint>
-  <joint name="kinect_yaw_joint" type="revolute">
-    <parent link="kurtana_pitch_link" />
-    <child link="kurtana_yaw_link" />
-    <origin xyz="0 0 0" rpy="0 0 0"/>
-    <axis xyz="0 1 0"/>
-    <limit effort="1000.0" lower="${-M_PI/2}" upper="${M_PI/2}" velocity="2.0"/>
-  </joint>
-  <include filename="$(find kurt_description)/parts/kinect.urdf.xacro" />
+  <include filename="$(find uos_common_urdf)/urdf/kinect.urdf.xacro" />
   <xacro:kinect camera="kinect" />
   <joint name="calvin_kinect_joint" type="fixed">
-    <parent link="kurtana_pitchpole_link" />
+    <parent link="kinect_yaw_link" />
     <child  link="kinect_link" />
-    <origin xyz="0.1 0 0.5" rpy="0 0.5 0"/>
+    <origin xyz="0.05 0 0" rpy="0 0.5 0"/>
   </joint>
-  <link name="kurtana_pitchpole_link">
-    <visual>
-      <origin rpy="${-M_PI/2} 0 0" xyz="0 0 0"/>
-      <geometry>
-        <cylinder radius="${pitchpole_radius}" length="${pitchpole_length}"/>
-      </geometry>
-      <material name="grey" />
-    </visual>
-    <collision>
-      <origin rpy="${-M_PI/2} 0 0" xyz="0 0 0"/>
-      <geometry>
-        <cylinder radius="${pitchpole_radius}" length="${pitchpole_length}"/>
-      </geometry>
-    </collision>
-    <xacro:cylinder_inertial radius="${pitchpole_radius}" length="${pitchpole_length}" mass="${pitchpole_mass}" />
-  </link>
   <xacro:macro name="kinect_pole_transmission" params="name">
     <transmission name="${name}_trans" type="pr2_mechanism_model/SimpleTransmission">
@@ -150,6 +154,5 @@
     </transmission>
   </xacro:macro>
-  <xacro:kinect_pole_transmission name="kinect_stretch" />
-  <xacro:kinect_pole_transmission name="kinect_roll" />
   <xacro:kinect_pole_transmission name="kinect_pitch" />
+  <xacro:kinect_pole_transmission name="kinect_yaw" />
 </robot>

Commit message: fix typo
this is not kurtana anymore

File: calvin_description/robots/calvin.urdf.xacro (robot description, xacro)
@@ -188,5 +188,5 @@
   </joint>
   <property name="baseplate_height" value="0.006" />
-  <joint name="kurtana_baseplate_controlbox_joint" type="fixed">
+  <joint name="calvin_baseplate_controlbox_joint" type="fixed">
     <parent link="structure" />
     <child link="katana_internal_controlbox_link" />

Commit message: Fuse urdf/calvin.urdf.xacro into robots/calvin.urdf.xacro

File: calvin_description/robots/calvin.urdf.xacro (robot description, xacro)
@@ -2,12 +2,242 @@
 <robot
   xmlns:xacro="http://ros.org/wiki/xacro"
+  xmlns:sensor="http://playerstage.sourceforge.net/gazebo/xmlschema/#sensor"
+  xmlns:controller="http://playerstage.sourceforge.net/gazebo/xmlschema/#controller"
   name="calvin">
   <include filename="$(find uos_common_urdf)/urdf/imu.gazebo.urdf.xacro" />
   <xacro:property name="imu_stdev" value="0.00017" />
   <include filename="$(find volksbot_driver)/urdf/volksbot.urdf.xacro" />
-  <include filename="$(find calvin_description)/urdf/calvin.urdf.xacro" />
-  <!--<include filename="$(find calvin_description)/urdf/gazebo.urdf.xacro" />-->
+  <property name="kinect_x_offset" value="0.06" />
+  <property name="kinect_y_offset" value="0.03" />
+  <property name="kinect_z_offset" value="0.05" />
+  <xacro:property name="pole_length" value="0.02"/>
+  <xacro:property name="pole_width" value="0.02"/>
+  <xacro:property name="pole_height" value="1"/>
+  <xacro:property name="structure_length" value="0.36"/>
+  <xacro:property name="structure_width" value="0.32"/>
+  <xacro:property name="structure_height" value="0.51"/>
+  <xacro:property name="item_width" value="0.02"/>
+  <xacro:property name="webcam_pitch_link_length" value="0.082"/>
+  <xacro:property name="webcam_pitch_link_width" value="0.095"/>
+  <xacro:property name="webcam_pitch_link_height" value="0.02"/>
+  <xacro:property name="webcam_z_offset" value="0.315"/>
+  <xacro:property name="kinect_pitch_link_length" value="0.08"/>
+  <xacro:property name="kinect_pitch_link_width" value="0.17"/>
+  <xacro:property name="kinect_pitch_link_height" value="0.02"/>
+  <xacro:property name="kinect_pitch_link_z_offset" value="0.46"/>
+  <link name="structure">
+    <visual>
+      <geometry>
+        <!--<box size="${structure_length} ${structure_width} ${structure_height}" />-->
+        <mesh filename="package://calvin_description/meshes/item-structure.stl"/>
+      </geometry>
+      <material name="grey" >
+        <color rgba="0.5 0.5 0.5 1" />
+      </material>
+    </visual>
+    <collision>
+      <geometry>
+        <!-- using STL for collision to fix http://answers.ros.org/question/2368/gazebo-model-wheels-slip-after-upgrade-to-electric -->
+        <!--<box size="${structure_length} ${structure_width} ${structure_height}" />-->
+        <mesh filename="package://calvin_description/meshes/item-structure.stl"/>
+      </geometry>
+    </collision>
+    <xacro:box_inertial x="${structure_length}" y="${structure_width}" z="${structure_height}" mass="2"/>
+  </link>
+  <joint name="top_to_structure" type="fixed">
+    <parent link="base_link" />
+    <child link="structure" />
+    <origin xyz="${base_link_length/2 - structure_length/2 - item_width} 0 ${structure_height/2 + base_link_height/2}" rpy="0 0 0" />
+  </joint>
+  <link name="imu" />
+  <joint name="structure_to_imu_joint" type="fixed">
+    <parent link="base_link" />
+    <child link="imu" />
+    <origin xyz="0 0 0" rpy="${M_PI} 0 ${M_PI}" />
+  </joint>
+  <link name="pole">
+    <visual>
+      <geometry>
+        <!--<box size="${pole_length} ${pole_width} ${pole_height}" />-->
+        <mesh filename="package://calvin_description/meshes/item-pole.stl"/>
+      </geometry>
+      <material name="grey" >
+        <color rgba="0.5 0.5 0.5 1" />
+      </material>
+    </visual>
+    <collision>
+      <geometry>
+        <!-- using STL for collision to fix http://answers.ros.org/question/2368/gazebo-model-wheels-slip-after-upgrade-to-electric -->
+        <!--<box size="${pole_length} ${pole_width} ${pole_height}" />-->
+        <mesh filename="package://calvin_description/meshes/item-pole.stl"/>
+      </geometry>
+    </collision>
+    <xacro:box_inertial x="${pole_length}" y="${pole_width}" z="${pole_height}" mass="0.25"/>
+  </link>
+  <joint name="structure_to_pole_joint" type="fixed">
+    <parent link="structure" />
+    <child link="pole" />
+    <origin xyz="${-structure_length/2 - pole_length/2} 0 ${pole_height/2 + structure_height/2}" rpy="0 0 0" />
+  </joint>
+  <!-- ******************************** -->
+  <!-- *** Sick_LMS200 Laser Scanner *** -->
+  <!-- ******************************** -->
+  <include filename="$(find uos_common_urdf)/urdf/sick_lms200.urdf.xacro" />
+  <xacro:sick_lms200 laser_link="sick_lms200" />
+  <joint name="structure_to_sick_lms200_joint" type="fixed" >
+    <parent link="structure" />
+    <child link="sick_lms200" />
+    <origin xyz="${-base_link_length/2 + structure_length/2 + item_width} 0 ${-structure_height/2 - base_link_height/2+0.18}" rpy="0 0 0" />
+  </joint>
+  <!-- ******************************** -->
+  <!-- *** gazebo ros camera plugin *** -->
+  <!-- ******************************** -->
+  <xacro:macro name="webcam" params="camera_name frame_prefix">
+    <gazebo reference="${frame_prefix}_link">
+      <sensor:camera name="${frame_prefix}_sensor">
+        <imageFormat>R8G8B8</imageFormat>
+        <imageSize>640 480</imageSize>
+        <hfov>45</hfov>
+        <nearClip>0.1</nearClip>
+        <farClip>100</farClip>
+        <updateRate>20.0</updateRate>
+        <controller:gazebo_ros_prosilica name="${frame_prefix}_controller" plugin="libgazebo_ros_prosilica.so">
+          <alwaysOn>true</alwaysOn>
+          <updateRate>20.0</updateRate>
+          <cameraName>${camera_name}</cameraName>
+          <imageTopicName>image_raw</imageTopicName>
+          <cameraInfoTopicName>camera_info</cameraInfoTopicName>
+          <frameName>${frame_prefix}_optical_link</frameName>
+          <CxPrime>1224.5</CxPrime>
+          <Cx>1224.5</Cx>
+          <Cy>1025.5</Cy>
+          <focalLength>772.548512</focalLength> <!-- image_width / (2*tan(hfov_radian /2)) -->
+          <distortionK1>0.0</distortionK1>
+          <distortionK2>0.0</distortionK2>
+          <distortionK3>0.0</distortionK3>
+          <distortionT1>0.0</distortionT1>
+          <distortionT2>0.0</distortionT2>
+        </controller:gazebo_ros_prosilica>
+      </sensor:camera>
+      <material value="Gazebo/Black" />
+    </gazebo>
+    <joint name="${frame_prefix}_pitch_joint" type="revolute">
+      <origin xyz="0 0 ${webcam_z_offset}" rpy="0 0 0" />
+      <parent link="pole" />
+      <child link="${frame_prefix}_pitch_link" />
+      <axis xyz="0 1 0"/>
+      <limit effort="1000.0" lower="${-M_PI/2}" upper="${M_PI/2}" velocity="2.0"/>
+    </joint>
+    <link name="${frame_prefix}_pitch_link">
+      <visual>
+        <origin rpy="0 0 0" xyz="${webcam_pitch_link_length/2 - item_width/2} 0 -${webcam_pitch_link_height}"/>
+        <geometry>
+          <box size="${webcam_pitch_link_length} ${webcam_pitch_link_width} ${webcam_pitch_link_height}" />
+        </geometry>
+        <material name="grey" >
+          <color rgba="0.5 0.5 0.5 1" />
+        </material>
+      </visual>
+      <collision>
+        <geometry>
+          <box size="${webcam_pitch_link_length} ${webcam_pitch_link_width} ${webcam_pitch_link_height}" />
+        </geometry>
+      </collision>
+      <xacro:box_inertial x="${webcam_pitch_link_length}" y="${webcam_pitch_link_width}" z="${webcam_pitch_link_height}" mass="0.01"/>
+    </link>
+    <joint name="${frame_prefix}_joint" type="fixed">
+      <origin xyz="0.06 0.01 -0.04" rpy="0 0 0" />
+      <parent link="${frame_prefix}_pitch_link" />
+      <child link="${frame_prefix}_link" />
+    </joint>
+    <link name="${frame_prefix}_link">
+      <visual>
+        <geometry>
+          <box size="0.02 0.085 0.02" />
+        </geometry>
+        <material name="black" >
+          <color rgba="0 0 0 1" />
+        </material>
+      </visual>
+      <collision>
+        <geometry>
+          <box size="0.02 0.085 0.02" />
+        </geometry>
+      </collision>
+      <xacro:box_inertial x="0.1" y="0.1" z="0.1" mass="0.01"/>
+    </link>
+    <joint name="${frame_prefix}_optical_joint" type="fixed">
+      <origin xyz="0 0 0" rpy="${-M_PI/2} 0 ${-M_PI/2}" />
+      <parent link="${frame_prefix}_link" />
+      <child link="${frame_prefix}_optical_link" />
+    </joint>
+    <link name="${frame_prefix}_optical_link">
+      <xacro:box_inertial x="0.1" y="0.1" z="0.1" mass="0.01"/>
+    </link>
+  </xacro:macro>
+  <xacro:webcam camera_name="webcam" frame_prefix="webcam" />
+  <!-- **************************** -->
+  <!-- *** Neuronics Katana Arm *** -->
+  <!-- **************************** -->
+  <include filename="$(find katana_description)/urdf/katana_450_6m90a_with_controlbox.urdf.xacro" />
+  <link name="katana_pattern"></link>
+  <joint name="katana_pattern_joint" type="fixed">
+    <parent link="katana_motor4_lift_link"/>
+    <child  link="katana_pattern" />
+    <origin xyz=".075 -.035 0.00" rpy="1.571 -1.571 0.151"/>
+  </joint>
+  <property name="baseplate_height" value="0.006" />
+  <joint name="kurtana_baseplate_controlbox_joint" type="fixed">
+    <parent link="structure" />
+    <child link="katana_internal_controlbox_link" />
+    <origin xyz="0 0 ${baseplate_height*1.5 + 0.2525}" rpy="0 0 0" />
+  </joint>
+  <!-- ********************************** -->
+  <!-- *** Kinect / Xtion RGBD Camera *** -->
+  <!-- ********************************** -->
+  <link name="kinect_pitch_link">
+    <visual>
+      <origin xyz="${kinect_pitch_link_length/2 - item_width/2} 0 0" rpy="0 0 0"/>
+      <geometry>
+        <box size="${kinect_pitch_link_length} ${kinect_pitch_link_width} ${kinect_pitch_link_height}" />
+      </geometry>
+      <material name="grey">
+        <color rgba="0.5 0.5 0.5 1" />
+      </material>
+    </visual>
+    <collision>
+      <origin xyz="${kinect_pitch_link_length/2 - item_width/2} 0 0" rpy="0 0 0"/>
+      <geometry>
+        <box size="${kinect_pitch_link_length} ${kinect_pitch_link_width} ${kinect_pitch_link_height}" />
+      </geometry>
+    </collision>
+    <xacro:box_inertial x="${kinect_pitch_link_length}" y="${kinect_pitch_link_width}" z="${kinect_pitch_link_height}" mass="0.01"/>
+  </link>
+  <joint name="kinect_pitch_joint" type="revolute">
+    <parent link="pole" />
+    <child link="kinect_pitch_link" />
+    <origin xyz="0 0 ${kinect_pitch_link_z_offset}" rpy="0 0 0"/>
+    <axis xyz="0 1 0"/>
+    <limit effort="1000.0" lower="${-M_PI/2}" upper="${M_PI/2}" velocity="2.0"/>
+  </joint>
+  <include filename="$(find uos_common_urdf)/urdf/kinect.urdf.xacro" />
+  <xacro:kinect camera="kinect" />
+  <joint name="calvin_kinect_joint" type="fixed">
+    <parent link="kinect_pitch_link" />
+    <child  link="kinect_link" />
+    <origin xyz="${kinect_x_offset} ${kinect_y_offset} ${kinect_z_offset}" rpy="0 0 0"/>
+  </joint>
+  <xacro:macro name="kinect_pole_transmission" params="name">
+    <transmission name="${name}_trans" type="pr2_mechanism_model/SimpleTransmission">
+      <actuator name="${name}_motor" />
+      <joint name="${name}_joint" />
+      <mechanicalReduction>1</mechanicalReduction>
+      <motorTorqueConstant>1</motorTorqueConstant>
+    </transmission>
+  </xacro:macro>
+  <xacro:kinect_pole_transmission name="kinect_pitch" />
+  <xacro:kinect_pole_transmission name="webcam_pitch" />
   <!-- inertial measurement unit for gazebo -->
-  <xacro:imu_gazebo link="base_link" imu_topic="imu" update_rate="100.0" stdev="${imu_stdev}" />
+  <xacro:imu_gazebo link="imu" imu_topic="imu" update_rate="100.0" stdev="${imu_stdev}" />
   <include filename="$(find sick_tim3xx)/urdf/sick_tim3xx.urdf.xacro" />
   <xacro:sick_tim3xx laser_link="laser" />

Commit message: calvin_description: rotated rgbd-cam in the urdf
Mounted an other rgbd-cam onto the robot that is mounted upside down, so the urdf had to be updated.

File: calvin_description/robots/calvin.urdf.xacro (robot description, xacro)
@@ -241,5 +241,5 @@
     <parent link="kinect_pitch_link" />
     <child  link="kinect_link" />
-    <origin xyz="${kinect_x_offset} ${kinect_y_offset} ${kinect_z_offset}" rpy="0 0 0"/>
+    <origin xyz="${kinect_x_offset} ${kinect_y_offset} ${kinect_z_offset}" rpy="${M_PI} 0 0"/>
   </joint>
   <xacro:macro name="kinect_pole_transmission" params="name">

Commit message: muffinhalterung/cup added to calvin

File: calvin_description/robots/calvin.urdf.xacro (robot description, xacro)
@@ -14,4 +14,6 @@
   <xacro:property name="pole_width" value="0.02"/>
   <xacro:property name="pole_height" value="1"/>
+  <xacro:property name="cup_radius" value="0.045"/>
+  <xacro:property name="cup_height" value="0.02"/>
   <xacro:property name="structure_length" value="0.36"/>
   <xacro:property name="structure_width" value="0.32"/>
@@ -79,4 +81,28 @@
     <child link="pole" />
     <origin xyz="${-structure_length/2 - pole_length/2} 0 ${pole_height/2 + structure_height/2}" rpy="0 0 0" />
+  </joint>
+  <link name="cup">
+    <visual>
+      <geometry>
+        <!--<cylinder length="${cup_height}" radius="${cup_radius}" />-->
+        <mesh filename="package://calvin_description/meshes/cup.stl"/>
+      </geometry>
+      <material name="grey" >
+        <color rgba="0.5 0.5 0.5 1" />
+      </material>
+    </visual>
+    <collision>
+      <geometry>
+        <!-- using STL for collision to fix http://answers.ros.org/question/2368/gazebo-model-wheels-slip-after-upgrade-to-electric -->
+        <!--<cylinder length="${cup_height}" radius="${cup_radius}" />-->
+        <mesh filename="package://calvin_description/meshes/cup.stl"/>
+      </geometry>
+    </collision>
+    <xacro:cylinder_inertial radius="${cup_radius}" length="${cup_height}" mass="0.05"/>
+  </link>
+  <joint name="structure_to_cup_joint" type="fixed">
+    <parent link="structure" />
+    <child link="cup" />
+    <origin xyz="${structure_length/2 - cup_radius} ${structure_width/2 - cup_radius} ${cup_height/2 + structure_height/2}" rpy="0 0 0" />
   </joint>
   <!-- ******************************** -->

Commit message: calvin_description: fixed urdf
Rotated the rgbd-cam in the urdf, because it was rotated in the so called real life.

File: calvin_description/robots/calvin.urdf.xacro (robot description, xacro)
@@ -226,5 +226,5 @@
     <parent link="kinect_pitch_link" />
     <child  link="kinect_link" />
-    <origin xyz="${kinect_x_offset} ${kinect_y_offset} ${kinect_z_offset}" rpy="0 0 0"/>
+    <origin xyz="${kinect_x_offset} ${kinect_y_offset} ${kinect_z_offset}" rpy="${M_PI} 0 0"/>
   </joint>
   <xacro:macro name="kinect_pole_transmission" params="name">

Commit message: calvin_description: fix inertials of webcam_link, webcam_optical_link
* webcam_link inertials now match collision dimensions
* webcam_optical_link doesn't need an inertial any more (no more
  Gazebo warnings in Hydro)

File: calvin_description/robots/calvin.urdf.xacro (robot description, xacro)
@@ -165,5 +165,5 @@
         </geometry>
       </collision>
-      <xacro:box_inertial x="0.1" y="0.1" z="0.1" mass="0.01"/>
+      <xacro:box_inertial x="0.02" y="0.085" z="0.02" mass="0.01"/>
     </link>
     <joint name="${frame_prefix}_optical_joint" type="fixed">
@@ -172,7 +172,5 @@
       <child link="${frame_prefix}_optical_link" />
     </joint>
-    <link name="${frame_prefix}_optical_link">
-      <xacro:box_inertial x="0.1" y="0.1" z="0.1" mass="0.01"/>
-    </link>
+    <link name="${frame_prefix}_optical_link" />
   </xacro:macro>
   <xacro:webcam camera_name="webcam" frame_prefix="webcam" />
