Commit message: calvin_description: fix inertials of webcam_link, webcam_optical_link
* webcam_link inertials now match collision dimensions
* webcam_optical_link doesn't need an inertial any more (no more
  Gazebo warnings in Hydro)

File: calvin_description/robots/calvin.urdf.xacro (robot description, xacro)
@@ -206,5 +206,5 @@
         </geometry>
       </collision>
-      <xacro:box_inertial x="0.1" y="0.1" z="0.1" mass="0.01"/>
+      <xacro:box_inertial x="0.02" y="0.085" z="0.02" mass="0.01"/>
     </link>
     <joint name="${frame_prefix}_optical_joint" type="fixed">
@@ -213,7 +213,5 @@
       <child link="${frame_prefix}_optical_link" />
     </joint>
-    <link name="${frame_prefix}_optical_link">
-      <xacro:box_inertial x="0.1" y="0.1" z="0.1" mass="0.01"/>
-    </link>
+    <link name="${frame_prefix}_optical_link" />
   </xacro:macro>
   <xacro:webcam camera_name="webcam" frame_prefix="webcam" />

Commit message: calvin_description: fixed inertials with origin

File: calvin_description/robots/calvin.urdf.xacro (robot description, xacro)
@@ -8,4 +8,5 @@
   <xacro:property name="imu_stdev" value="0.00017" />
   <xacro:include filename="$(find volksbot_driver)/urdf/volksbot.urdf.xacro" />
+  <xacro:include filename="$(find uos_common_urdf)/common.xacro" />
   <property name="kinect_x_offset" value="0.07" />
   <property name="kinect_y_offset" value="-0.02" />
@@ -181,9 +182,12 @@
       </visual>
       <collision>
+        <origin rpy="0 0 0" xyz="${webcam_pitch_link_length/2 - item_width/2} 0 -${webcam_pitch_link_height}"/>
         <geometry>
           <box size="${webcam_pitch_link_length} ${webcam_pitch_link_width} ${webcam_pitch_link_height}" />
         </geometry>
       </collision>
-      <xacro:box_inertial x="${webcam_pitch_link_length}" y="${webcam_pitch_link_width}" z="${webcam_pitch_link_height}" mass="0.01"/>
+      <xacro:box_inertial_with_origin x="${webcam_pitch_link_length}" y="${webcam_pitch_link_width}" z="${webcam_pitch_link_height}" mass="0.01">
+        <origin rpy="0 0 0" xyz="${webcam_pitch_link_length/2 - item_width/2} 0 -${webcam_pitch_link_height}"/>
+      </xacro:box_inertial_with_origin>
     </link>
     <joint name="${frame_prefix}_joint" type="fixed">
@@ -251,5 +255,7 @@
       </geometry>
     </collision>
-    <xacro:box_inertial x="${kinect_pitch_link_length}" y="${kinect_pitch_link_width}" z="${kinect_pitch_link_height}" mass="0.01"/>
+    <xacro:box_inertial_with_origin x="${kinect_pitch_link_length}" y="${kinect_pitch_link_width}" z="${kinect_pitch_link_height}" mass="0.01">
+      <origin xyz="${kinect_pitch_link_length/2 - item_width/2} 0 0" rpy="0 0 0"/>
+    </xacro:box_inertial_with_origin>
   </link>
   <joint name="kinect_pitch_joint" type="revolute">

Commit message: calvin_description: fixed inertials with origin
Conflicts:
	calvin_description/robots/calvin.urdf.xacro

File: calvin_description/robots/calvin.urdf.xacro (robot description, xacro)
@@ -8,4 +8,5 @@
   <xacro:property name="imu_stdev" value="0.00017" />
   <include filename="$(find volksbot_driver)/urdf/volksbot.urdf.xacro" />
+  <include filename="$(find uos_common_urdf)/common.xacro" />
   <property name="kinect_x_offset" value="0.06" />
   <property name="kinect_y_offset" value="0.03" />
@@ -140,9 +141,12 @@
       </visual>
       <collision>
+        <origin rpy="0 0 0" xyz="${webcam_pitch_link_length/2 - item_width/2} 0 -${webcam_pitch_link_height}"/>
         <geometry>
           <box size="${webcam_pitch_link_length} ${webcam_pitch_link_width} ${webcam_pitch_link_height}" />
         </geometry>
       </collision>
-      <xacro:box_inertial x="${webcam_pitch_link_length}" y="${webcam_pitch_link_width}" z="${webcam_pitch_link_height}" mass="0.01"/>
+      <xacro:box_inertial_with_origin x="${webcam_pitch_link_length}" y="${webcam_pitch_link_width}" z="${webcam_pitch_link_height}" mass="0.01">
+        <origin rpy="0 0 0" xyz="${webcam_pitch_link_length/2 - item_width/2} 0 -${webcam_pitch_link_height}"/>
+      </xacro:box_inertial_with_origin>
     </link>
     <joint name="${frame_prefix}_joint" type="fixed">
@@ -210,5 +214,7 @@
       </geometry>
     </collision>
-    <xacro:box_inertial x="${kinect_pitch_link_length}" y="${kinect_pitch_link_width}" z="${kinect_pitch_link_height}" mass="0.01"/>
+    <xacro:box_inertial_with_origin x="${kinect_pitch_link_length}" y="${kinect_pitch_link_width}" z="${kinect_pitch_link_height}" mass="0.01">
+      <origin xyz="${kinect_pitch_link_length/2 - item_width/2} 0 0" rpy="0 0 0"/>
+    </xacro:box_inertial_with_origin>
   </link>
   <joint name="kinect_pitch_joint" type="revolute">

Commit message: calvin_description: calibrated the laser scanners on the xy-plane
Calibrated the big laser scanner against the tiny scanner on the x-axis by hand.
Moved the tiny laser scanner on the y-axis, because it is not in the middle of calvin on the y-axis.

File: calvin_description/robots/calvin.urdf.xacro (robot description, xacro)
@@ -89,5 +89,5 @@
     <parent link="structure" />
     <child link="sick_lms200" />
-    <origin xyz="${-base_link_length/2 + structure_length/2 + item_width} 0 ${-structure_height/2 - base_link_height/2+0.18}" rpy="0 0 0" />
+    <origin xyz="${-base_link_length/2 + structure_length/2 + item_width - 0.015} 0 ${-structure_height/2 - base_link_height/2+0.18}" rpy="0 0 0" />
   </joint>
   <!-- ******************************** -->
@@ -247,5 +247,5 @@
   <xacro:sick_tim3xx laser_link="laser" />
   <joint name="laser_mount_joint" type="fixed">
-    <origin xyz="0.25 0 0.08" rpy="0 0 0" />
+    <origin xyz="0.25 0.0035 0.08" rpy="0 0 0" />
     <parent link="base_link"/>
     <child link="laser_mount_link" />

Commit message: calvin_description: calibrated the laser scanners on the xy-plane
Calibrated the big laser scanner against the tiny scanner on the x-axis by hand.
Moved the tiny laser scanner on the y-axis, because it is not in the middle of calvin on the y-axis.

File: calvin_description/robots/calvin.urdf.xacro (robot description, xacro)
@@ -115,5 +115,5 @@
     <parent link="structure" />
     <child link="sick_lms200" />
-    <origin xyz="${-base_link_length/2 + structure_length/2 + item_width} 0 ${-structure_height/2 - base_link_height/2+0.18}" rpy="0 0 0" />
+    <origin xyz="${-base_link_length/2 + structure_length/2 + item_width - 0.015} 0 ${-structure_height/2 - base_link_height/2+0.18}" rpy="0 0 0" />
   </joint>
   <!-- ******************************** -->
@@ -290,5 +290,5 @@
   <xacro:sick_tim3xx laser_link="laser" />
   <joint name="laser_mount_joint" type="fixed">
-    <origin xyz="0.25 0 0.08" rpy="0 0 0" />
+    <origin xyz="0.25 0.0035 0.08" rpy="0 0 0" />
     <parent link="base_link"/>
     <child link="laser_mount_link" />

Commit message: calvin_description: replaced buggy camera_plugin for vgacam with the one for kinect/xtion
messy fix with several unnecessary topics, but does the trick for now.

File: calvin_description/robots/calvin.urdf.xacro (robot description, xacro)
@@ -122,5 +122,5 @@
   <xacro:macro name="webcam" params="camera_name frame_prefix">
     <gazebo reference="${frame_prefix}_link">
-      <sensor type="camera" name="${frame_prefix}_sensor">
+      <sensor type="depth" name="${frame_prefix}_sensor">
         <always_on>true</always_on>
         <update_rate>20.0</update_rate>
@@ -138,9 +138,20 @@
           </clip>
         </camera>
-        <plugin name="${frame_prefix}_plugin" filename="libgazebo_ros_camera.so">
+        <plugin name="${frame_prefix}_plugin" filename="libgazebo_ros_openni_kinect.so">
+          <alwaysOn>true</alwaysOn>
+          <updateRate>1.0</updateRate>
           <cameraName>${camera_name}</cameraName>
           <imageTopicName>image_raw</imageTopicName>
           <cameraInfoTopicName>camera_info</cameraInfoTopicName>
+          <depthImageTopicName>/${camera_name}/depth/image_raw</depthImageTopicName>
+          <depthImageCameraInfoTopicName>/${camera_name}/depth/camera_info</depthImageCameraInfoTopicName>
+          <pointCloudTopicName>/${camera_name}/depth_registered/points</pointCloudTopicName>
+          <pointCloudCutoff>0.5</pointCloudCutoff>
           <frameName>${frame_prefix}_optical_link</frameName>
+          <distortionK1>0.0</distortionK1>
+          <distortionK2>0.0</distortionK2>
+          <distortionK3>0.0</distortionK3>
+          <distortionT1>0.0</distortionT1>
+          <distortionT2>0.0</distortionT2>
         </plugin>
 <!-- This keeps segfaulting on hydro, use gazebo_ros_camera for now
@@ -170,4 +181,5 @@
       <axis xyz="0 1 0"/>
       <limit effort="1000.0" lower="${-M_PI/2}" upper="${M_PI/2}" velocity="2.0"/>
+      <dynamics damping="0.1"/>
     </joint>
     <link name="${frame_prefix}_pitch_link">
@@ -219,5 +231,5 @@
     <link name="${frame_prefix}_optical_link" />
   </xacro:macro>
-  <xacro:webcam camera_name="webcam" frame_prefix="webcam" />
+  <xacro:webcam camera_name="vgacam" frame_prefix="webcam" />
   <!-- **************************** -->
   <!-- *** Neuronics Katana Arm *** -->

Commit message: imu urdf position adjusted to real position

File: calvin_description/robots/calvin.urdf.xacro (robot description, xacro)
@@ -57,5 +57,5 @@
     <parent link="base_link" />
     <child link="imu" />
-    <origin xyz="0 0 0" rpy="${M_PI} 0 ${M_PI}" />
+    <origin xyz="-0.165 0.135 0.08" rpy="${M_PI} 0 ${M_PI}" />
   </joint>
   <link name="pole">

Commit message: calvin_description: calibrated the small laser scanner
Changed pitch and the position on the z-axis.

File: calvin_description/robots/calvin.urdf.xacro (robot description, xacro)
@@ -11,5 +11,5 @@
   <property name="kinect_x_offset" value="0.07" />
   <property name="kinect_y_offset" value="-0.02" />
-  <property name="kinect_z_offset" value="0.01" />
+  <property name="kinect_z_offset" value="0.0" />
   <xacro:property name="pole_length" value="0.02"/>
   <xacro:property name="pole_width" value="0.02"/>
@@ -302,5 +302,5 @@
   <xacro:sick_tim3xx laser_link="laser" />
   <joint name="laser_mount_joint" type="fixed">
-    <origin xyz="0.25 0.0035 0.08" rpy="0 0 0" />
+    <origin xyz="0.25 0.0035 ${0.264185 - 0.1275 - (0.32017 - 0.26419)}" rpy="0 -0.0604984 0" />
     <parent link="base_link"/>
     <child link="laser_mount_link" />

Commit message: calvin_description: calibrated the big laser scanner
Changed the pitch and the position on the z-axis.

File: calvin_description/robots/calvin.urdf.xacro (robot description, xacro)
@@ -115,5 +115,5 @@
     <parent link="structure" />
     <child link="sick_lms200" />
-    <origin xyz="${-base_link_length/2 + structure_length/2 + item_width - 0.015} 0 ${-structure_height/2 - base_link_height/2+0.18}" rpy="0 0 0" />
+    <origin xyz="${-base_link_length/2 + structure_length/2 + item_width - 0.015} 0 ${-0.46 + 0.297204}" rpy="0 -0.00809693 0" />
   </joint>
   <!-- ******************************** -->

Commit message: calvin_description: adapted the urdf to the new version of the volksbot urdf
The z-coordinate of base_link in the volksbot urdf is 3 mm heigher now.
The values of the z-coordinates of the laser scanners had to be adapted.
The calculation of the z-coordinate of the tiny laser scanner uses variables now.

File: calvin_description/robots/calvin.urdf.xacro (robot description, xacro)
@@ -115,5 +115,5 @@
     <parent link="structure" />
     <child link="sick_lms200" />
-    <origin xyz="${-base_link_length/2 + structure_length/2 + item_width - 0.015} 0 ${-0.46 + 0.297204}" rpy="0 -0.00809693 0" />
+    <origin xyz="${-base_link_length/2 + structure_length/2 + item_width - 0.015} 0 ${-0.463 + 0.297204}" rpy="0 -0.00809693 0" />
   </joint>
   <!-- ******************************** -->
@@ -301,5 +301,5 @@
   <xacro:sick_tim3xx laser_link="laser" />
   <joint name="laser_mount_joint" type="fixed">
-    <origin xyz="0.25 0.0035 ${0.264185 - 0.1275 - (0.32017 - 0.26419)}" rpy="0 -0.0604984 0" />
+    <origin xyz="0.25 0.0035 ${0.264185 - (wheel_radius - wheel_z_offset) - sick_tim3xx_z_offset}" rpy="0 -0.0604984 0" />
     <parent link="base_link"/>
     <child link="laser_mount_link" />

Commit message: calvin_description: using the new link "base_top" in the urdf

File: calvin_description/robots/calvin.urdf.xacro (robot description, xacro)
@@ -49,13 +49,13 @@
   </link>
   <joint name="top_to_structure" type="fixed">
-    <parent link="base_link" />
+    <parent link="base_top" />
     <child link="structure" />
-    <origin xyz="${base_link_length/2 - structure_length/2 - item_width} 0 ${structure_height/2 + base_link_height/2}" rpy="0 0 0" />
+    <origin xyz="${base_link_length/2 - structure_length/2 - item_width} 0 ${structure_height/2}" rpy="0 0 0" />
   </joint>
   <link name="imu" />
   <joint name="structure_to_imu_joint" type="fixed">
-    <parent link="base_link" />
+    <parent link="base_top" />
     <child link="imu" />
-    <origin xyz="-0.165 0.135 0.08" rpy="${M_PI} 0 ${M_PI}" />
+    <origin xyz="-0.165 0.135 0" rpy="${M_PI} 0 ${M_PI}" />
   </joint>
   <link name="pole">
@@ -301,6 +301,6 @@
   <xacro:sick_tim3xx laser_link="laser" />
   <joint name="laser_mount_joint" type="fixed">
-    <origin xyz="0.25 0.0035 ${0.264185 - (wheel_radius - wheel_z_offset) - sick_tim3xx_z_offset}" rpy="0 -0.0604984 0" />
-    <parent link="base_link"/>
+    <origin xyz="0.25 0.0035 ${0.264185 - (wheel_radius - wheel_z_offset + base_link_height / 2.0) - sick_tim3xx_z_offset}" rpy="0 -0.0604984 0" />
+    <parent link="base_top"/>
     <child link="laser_mount_link" />
   </joint>

Commit message: Revert "calvin_description: using the new link "base_top" in the urdf"
this completely fucked up push_button. like completely.

This reverts commit fa28a0cec9170216976574e7af4c4848e49e70d9.

Conflicts:

	calvin_description/robots/calvin.urdf.xacro

File: calvin_description/robots/calvin.urdf.xacro (robot description, xacro)
@@ -49,13 +49,13 @@
   </link>
   <joint name="top_to_structure" type="fixed">
-    <parent link="base_top" />
+    <parent link="base_link" />
     <child link="structure" />
-    <origin xyz="${base_link_length/2 - structure_length/2 - item_width} 0 ${structure_height/2}" rpy="0 0 0" />
+    <origin xyz="${base_link_length/2 - structure_length/2 - item_width} 0 ${structure_height/2 + base_link_height/2}" rpy="0 0 0" />
   </joint>
   <link name="imu" />
   <joint name="structure_to_imu_joint" type="fixed">
-    <parent link="base_top" />
+    <parent link="base_link" />
     <child link="imu" />
-    <origin xyz="-0.165 0.135 0" rpy="${M_PI} 0 ${M_PI}" />
+    <origin xyz="-0.165 0.135 0.08" rpy="${M_PI} 0 ${M_PI}" />
   </joint>
   <link name="pole">
@@ -301,9 +301,6 @@
   <xacro:sick_tim3xx laser_link="laser" />
   <joint name="laser_mount_joint" type="fixed">
-    <!-- 0.264185 is the z-coordinate of the laser scanner measured from the ground
-         (wheel_radius - wheel_z_offset + base_link_height / 2.0) is the z-coordinate of base_top
-         sick_tim3xx_z_offset is the difference in the z-position between the laser_mount_link and the actual laser scanner -->
-    <origin xyz="0.25 0.0035 ${0.264185 - (wheel_radius - wheel_z_offset + base_link_height / 2.0) - sick_tim3xx_z_offset}" rpy="0 -0.0604984 0" />
-    <parent link="base_top"/>
+    <origin xyz="0.25 0.0035 ${0.264185 - (wheel_radius - wheel_z_offset) - sick_tim3xx_z_offset}" rpy="0 -0.0604984 0" />
+    <parent link="base_link"/>
     <child link="laser_mount_link" />
   </joint>

Commit message: Revert "Revert "calvin_description: using the new link "base_top" in the urdf""
This reverts commit 50de6b4dc9364c3df45c99704195e50f10af1c4b. Fixed now
in push_button.

File: calvin_description/robots/calvin.urdf.xacro (robot description, xacro)
@@ -49,13 +49,13 @@
   </link>
   <joint name="top_to_structure" type="fixed">
-    <parent link="base_link" />
+    <parent link="base_top" />
     <child link="structure" />
-    <origin xyz="${base_link_length/2 - structure_length/2 - item_width} 0 ${structure_height/2 + base_link_height/2}" rpy="0 0 0" />
+    <origin xyz="${base_link_length/2 - structure_length/2 - item_width} 0 ${structure_height/2}" rpy="0 0 0" />
   </joint>
   <link name="imu" />
   <joint name="structure_to_imu_joint" type="fixed">
-    <parent link="base_link" />
+    <parent link="base_top" />
     <child link="imu" />
-    <origin xyz="-0.165 0.135 0.08" rpy="${M_PI} 0 ${M_PI}" />
+    <origin xyz="-0.165 0.135 0" rpy="${M_PI} 0 ${M_PI}" />
   </joint>
   <link name="pole">
@@ -301,6 +301,9 @@
   <xacro:sick_tim3xx laser_link="laser" />
   <joint name="laser_mount_joint" type="fixed">
-    <origin xyz="0.25 0.0035 ${0.264185 - (wheel_radius - wheel_z_offset) - sick_tim3xx_z_offset}" rpy="0 -0.0604984 0" />
-    <parent link="base_link"/>
+    <!-- 0.264185 is the z-coordinate of the laser scanner measured from the ground
+         (wheel_radius - wheel_z_offset + base_link_height / 2.0) is the z-coordinate of base_top
+         sick_tim3xx_z_offset is the difference in the z-position between the laser_mount_link and the actual laser scanner -->
+    <origin xyz="0.25 0.0035 ${0.264185 - (wheel_radius - wheel_z_offset + base_link_height / 2.0) - sick_tim3xx_z_offset}" rpy="0 -0.0604984 0" />
+    <parent link="base_top"/>
     <child link="laser_mount_link" />
   </joint>

Commit message: calvin robot: adjusted webcam z offset

File: calvin_description/robots/calvin.urdf.xacro (robot description, xacro)
@@ -24,5 +24,5 @@
   <xacro:property name="webcam_pitch_link_width" value="0.095"/>
   <xacro:property name="webcam_pitch_link_height" value="0.02"/>
-  <xacro:property name="webcam_z_offset" value="0.315"/>
+  <xacro:property name="webcam_z_offset" value="0.412"/>
   <xacro:property name="kinect_pitch_link_length" value="0.08"/>
   <xacro:property name="kinect_pitch_link_width" value="0.17"/>

Commit message: calvin_description, calvin_joint_commander: calibrated new rgbd cam

File: calvin_description/robots/calvin.urdf.xacro (robot description, xacro)
@@ -9,5 +9,5 @@
   <xacro:include filename="$(find volksbot_driver)/urdf/volksbot.urdf.xacro" />
   <xacro:include filename="$(find uos_common_urdf)/common.xacro" />
-  <property name="kinect_x_offset" value="0.07" />
+  <property name="kinect_x_offset" value="0.09" />
   <property name="kinect_y_offset" value="-0.02" />
   <property name="kinect_z_offset" value="0.0" />
@@ -23,10 +23,10 @@
   <xacro:property name="webcam_pitch_link_length" value="0.082"/>
   <xacro:property name="webcam_pitch_link_width" value="0.095"/>
-  <xacro:property name="webcam_pitch_link_height" value="0.02"/>
+  <xacro:property name="webcam_pitch_link_height" value="0.04"/>
   <xacro:property name="webcam_z_offset" value="0.412"/>
   <xacro:property name="kinect_pitch_link_length" value="0.08"/>
   <xacro:property name="kinect_pitch_link_width" value="0.17"/>
-  <xacro:property name="kinect_pitch_link_height" value="0.02"/>
-  <xacro:property name="kinect_pitch_link_z_offset" value="0.46"/>
+  <xacro:property name="kinect_pitch_link_height" value="0.04"/>
+  <xacro:property name="kinect_pitch_link_z_offset" value="0.44"/>
   <link name="structure">
     <visual>

Commit message: calvin_description, calvin_joint_commander: updated values of the pole, webcam and kinect
Put the pole on the correct (new) position.
Changed the height of the pole in the urdf and the mesh.
Changed the position of the webcam and the kinect.
Changed the pitch of the kinect.
The yaw of the webcam and the kinect is still not correct.

File: calvin_description/robots/calvin.urdf.xacro (robot description, xacro)
@@ -14,5 +14,5 @@
   <xacro:property name="pole_length" value="0.02"/>
   <xacro:property name="pole_width" value="0.02"/>
-  <xacro:property name="pole_height" value="1"/>
+  <xacro:property name="pole_height" value="1.405"/>
   <xacro:property name="cup_radius" value="0.045"/>
   <xacro:property name="cup_height" value="0.02"/>
@@ -24,9 +24,9 @@
   <xacro:property name="webcam_pitch_link_width" value="0.095"/>
   <xacro:property name="webcam_pitch_link_height" value="0.04"/>
-  <xacro:property name="webcam_z_offset" value="0.412"/>
+  <xacro:property name="webcam_z_offset" value="0.61"/>
   <xacro:property name="kinect_pitch_link_length" value="0.08"/>
   <xacro:property name="kinect_pitch_link_width" value="0.17"/>
   <xacro:property name="kinect_pitch_link_height" value="0.04"/>
-  <xacro:property name="kinect_pitch_link_z_offset" value="0.44"/>
+  <xacro:property name="kinect_pitch_link_z_offset" value="0.66"/>
   <link name="structure">
     <visual>
@@ -81,5 +81,5 @@
     <parent link="structure" />
     <child link="pole" />
-    <origin xyz="${-structure_length/2 - pole_length/2} 0 ${pole_height/2 + structure_height/2}" rpy="0 0 0" />
+    <origin xyz="${-structure_length/2 - pole_length/2} 0 ${structure_height/2 + 0.3}" rpy="0 0 0" />
   </joint>
   <link name="cup">

Commit message: calvin_description, calvin_joint_commander: calibrated the webcam

File: calvin_description/robots/calvin.urdf.xacro (robot description, xacro)
@@ -24,5 +24,5 @@
   <xacro:property name="webcam_pitch_link_width" value="0.095"/>
   <xacro:property name="webcam_pitch_link_height" value="0.04"/>
-  <xacro:property name="webcam_z_offset" value="0.61"/>
+  <xacro:property name="webcam_z_offset" value="0.6"/>
   <xacro:property name="kinect_pitch_link_length" value="0.08"/>
   <xacro:property name="kinect_pitch_link_width" value="0.17"/>
@@ -175,5 +175,5 @@
     </gazebo>
     <joint name="${frame_prefix}_pitch_joint" type="revolute">
-      <origin xyz="0 0 ${webcam_z_offset}" rpy="0 0 0" />
+      <origin xyz="0 0 ${webcam_z_offset}" rpy="0 0 -0.029" />
       <parent link="pole" />
       <child link="${frame_prefix}_pitch_link" />

Commit message: calvin_description: calibrated rgbd cam

File: calvin_description/robots/calvin.urdf.xacro (robot description, xacro)
@@ -9,5 +9,5 @@
   <xacro:include filename="$(find volksbot_driver)/urdf/volksbot.urdf.xacro" />
   <xacro:include filename="$(find uos_common_urdf)/common.xacro" />
-  <property name="kinect_x_offset" value="0.09" />
+  <property name="kinect_x_offset" value="0.1" />
   <property name="kinect_y_offset" value="-0.02" />
   <property name="kinect_z_offset" value="0.0" />
@@ -28,5 +28,5 @@
   <xacro:property name="kinect_pitch_link_width" value="0.17"/>
   <xacro:property name="kinect_pitch_link_height" value="0.04"/>
-  <xacro:property name="kinect_pitch_link_z_offset" value="0.66"/>
+  <xacro:property name="kinect_pitch_link_z_offset" value="0.65"/>
   <link name="structure">
     <visual>
