Commit message: adjust to sick_tim3xx -> sick_tim rename

File: calvin_description/robots/calvin.urdf.xacro (robot description, xacro)
@@ -298,11 +298,11 @@
   <!-- inertial measurement unit for gazebo -->
   <xacro:imu_gazebo link="imu" imu_topic="imu/data" update_rate="100.0" stdev="${imu_stdev}" />
-  <xacro:include filename="$(find sick_tim3xx)/urdf/sick_tim3xx.urdf.xacro" />
-  <xacro:sick_tim3xx laser_link="laser" />
+  <xacro:include filename="$(find sick_tim)/urdf/sick_tim.urdf.xacro" />
+  <xacro:sick_tim310 name="laser" ros_topic="scan" />
   <joint name="laser_mount_joint" type="fixed">
     <!-- 0.264185 is the z-coordinate of the laser scanner measured from the ground
          (wheel_radius - wheel_z_offset + base_link_height / 2.0) is the z-coordinate of base_top
-         sick_tim3xx_z_offset is the difference in the z-position between the laser_mount_link and the actual laser scanner -->
-    <origin xyz="0.25 0.0035 ${0.264185 - (wheel_radius - wheel_z_offset + base_link_height / 2.0) - sick_tim3xx_z_offset}" rpy="0 -0.0604984 0" />
+         0.05595 (sick_tim z_offset) is the difference in the z-position between the laser_mount_link and the actual laser scanner -->
+    <origin xyz="0.25 0.0035 ${0.264185 - (wheel_radius - wheel_z_offset + base_link_height / 2.0) - 0.05595}" rpy="0 -0.0604984 0" />
     <parent link="base_top"/>
     <child link="laser_mount_link" />

Commit message: hardware interface is now a required option of transmission/joint
This change is not harmful with hydro and fixes the gazebo simulation with indigo

File: calvin_description/robots/calvin.urdf.xacro (robot description, xacro)
@@ -287,6 +287,8 @@
     <transmission name="${name}_trans">
       <type>transmission_interface/SimpleTransmission</type>
-      <joint name="${name}_joint" />
-      <actuator name="${name}_motor" >
+      <joint name="${name}_joint">
+        <hardwareInterface>EffortJointInterface</hardwareInterface>
+      </joint>
+      <actuator name="${name}_motor">
         <hardwareInterface>EffortJointInterface</hardwareInterface>
         <mechanicalReduction>1</mechanicalReduction>

Commit message: changed position from tim310 laserscan to the back of calvin

File: calvin_description/robots/calvin.urdf.xacro (robot description, xacro)
@@ -300,4 +300,7 @@
   <!-- inertial measurement unit for gazebo -->
   <xacro:imu_gazebo link="imu" imu_topic="imu/data" update_rate="100.0" stdev="${imu_stdev}" />
+  <!-- ******************************** -->
+  <!-- *** Sick_TIM Laser Scanner *** -->
+  <!-- ******************************** -->
   <xacro:include filename="$(find sick_tim)/urdf/sick_tim.urdf.xacro" />
   <xacro:sick_tim310 name="laser" ros_topic="scan" />
@@ -306,7 +309,13 @@
          (wheel_radius - wheel_z_offset + base_link_height / 2.0) is the z-coordinate of base_top
          0.05595 (sick_tim z_offset) is the difference in the z-position between the laser_mount_link and the actual laser scanner -->
-    <origin xyz="0.25 0.0035 ${0.264185 - (wheel_radius - wheel_z_offset + base_link_height / 2.0) - 0.05595}" rpy="0 -0.0604984 0" />
+    <origin xyz="-0.25 -0.008 ${0.264185 - (wheel_radius - wheel_z_offset + base_link_height / 2.0) - 0.05595}" rpy="0 -0.0504984 ${M_PI}" />
     <parent link="base_top"/>
     <child link="laser_mount_link" />
   </joint>
+  <link name="laser_center"/>
+  <joint name="base_top_to_laser_center" type="fixed">
+    <parent link="base_top"/>
+    <child link="laser_center"/>
+    <origin xyz="0 0 0.06" rpy="0 0 0"/>
+  </joint>
 </robot>

Commit message: adjust IMU position to reflect modified hardware

File: calvin_description/robots/calvin.urdf.xacro (robot description, xacro)
@@ -54,8 +54,8 @@
   </joint>
   <link name="imu" />
-  <joint name="structure_to_imu_joint" type="fixed">
-    <parent link="base_top" />
+  <joint name="base_link_to_imu_joint" type="fixed">
+    <parent link="base_link" />
     <child link="imu" />
-    <origin xyz="-0.165 0.135 0" rpy="${M_PI} 0 ${M_PI}" />
+    <origin xyz="${base_link_length/2 - .12} 0 -${base_link_height/2 - .01}" rpy="${M_PI} 0 ${M_PI/2}" />
   </joint>
   <link name="pole">

Commit message: add radar sensor to calvin urdf
This depends on the respective commit in uos_tools
that adds the inras_radar description.

File: calvin_description/robots/calvin.urdf.xacro (robot description, xacro)
@@ -319,3 +319,13 @@
     <origin xyz="0 0 0.06" rpy="0 0 0"/>
   </joint>
+  <!-- ************************** -->
+  <!-- *** INRAS Radar Sensor *** -->
+  <!-- ************************** -->
+  <xacro:include filename="$(find uos_common_urdf)/urdf/inras_radar.urdf.xacro" />
+  <xacro:inras_radar radar_link="radar" />
+  <joint name="structure_to_radar_joint" type="fixed">
+    <origin xyz="${structure_length/2 + radar_length - radar_center_x_pos} ${radar_center_y_pos - radar_width/2 } ${structure_height/2 + 0.023 - radar_height + radar_center_z_pos}" rpy="0 0 0" />
+    <parent link="structure" />
+    <child link="radar" />
+  </joint>
 </robot>
